File: board/t80-psu12.kicad_pcb (KiCad board)
At the start: 2 copper layers, 26 x 80 mm, 28 parts, among them J1 Conn_01x02_Female, U1 FR8205, U2 FR8205

Commit message: WIP
Parts:
- moved C1 1.00 mm to (106.0, 133.0)
- moved C7 1.00 mm to (106.0, 122.0)
- moved X2 1.00 mm to (106.1, 95.0)
- moved C3 0.50 mm to (103.5, 74.0)
- moved C4 0.50 mm to (91.5, 74.0)
- moved C5 0.50 mm to (104.5, 81.0)
- moved C6 0.50 mm to (92.5, 81.0)
- moved D1 0.50 mm to (97.5, 86.0)
- moved L1 0.50 mm to (103.5, 68.0)
- moved L2 0.50 mm to (91.5, 68.0)
- moved NT1 0.50 mm to (94.5, 95.0)
- moved NT2 0.50 mm to (100.5, 108.0)
- moved NT3 0.50 mm to (97.5, 105.0)
- moved NT4 0.50 mm to (91.5, 97.5)
- moved NT5 0.50 mm to (91.5, 97.5)
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Routing:
- net +5V: track 65.1 -> 63.3 mm
- net +12V: track 121.0 -> 119.3 mm
- net /PWR_LINE_12V: track 23.4 -> 22.3 mm
- net /SDA: track 21.8 -> 20.8 mm
- net /SCL: track 21.8 -> 20.8 mm
- net /IRQ: track 21.9 -> 20.9 mm
- net /RST: track 21.9 -> 20.9 mm
- net /PWR_LINE_GND: track 23.4 -> 22.4 mm
- net /PWR_LINE_5V: track 23.9 -> 23.2 mm
- net /PWR_LINE_3V3: track 23.9 -> 23.2 mm
Other:
- board size 26 x 80 mm -> 25 x 80 mm

Commit message: WIP
Parts:
- removed NT1, NT2, NT3, NT4, NT5: NetTie_2, t80:NetTie-2mm-T80
- removed X2: ~, Connector_PinHeader_2.54mm:PinHeader_2x05_P2.54mm_Vertical
- X1: footprint Connector_PinHeader_2.54mm:PinHeader_2x05_P2.54mm_Vertical -> Connector_IDC:IDC-Header_2x04_P2.54mm_Vertical
- moved C4 27.0 mm to (105.5, 95.0)
- moved C8 23.7 mm to (105.5, 105.0), turned to 90 degrees
- moved C2 17.7 mm to (89.0, 128.0), turned to -90 degrees
- moved C6 17.7 mm to (106.0, 128.0), turned to -90 degrees
- moved X1 2.34 mm to (88.3, 96.2)
- moved C1 1.00 mm to (103.5, 81.0)
- moved C5 1.00 mm to (91.5, 81.0)
- moved R6 0.51 mm to (100.5, 83.5)
- renumbered C5 to C1, C1 to C2, C7 to C4, C6 to C5, C2 to C6, C4 to C7, R2 to R1, R4 to R2, R5 to R3, R3 to R4, R6 to R5, R1 to R6
Connections:
- X1 pad 1: /PWR_LINE_12V -> GND
- X1 pad 2: /PWR_LINE_12V -> unconnected-(X1-SCL)
- X1 pad 3: /PWR_LINE_GND -> unconnected-(X1-SDA)
- X1 pad 4: /PWR_LINE_GND -> +3V3
- X1 pad 5: /SCL -> unconnected-(X1-RST)
- X1 pad 6: /SDA -> unconnected-(X1-IRQ)
- X1 pad 7: /RST -> GND
- X1 pad 8: /IRQ -> +5V
Routing:
- net GND: track 57.8 -> 25.9 mm
- net /PWR_LINE_5V: track 23.2 -> 0.00 mm, vias 1 -> 0
- net /PWR_LINE_3V3: track 23.2 -> 0.00 mm, vias 1 -> 0
- net /PWR_LINE_GND: track 22.4 -> 0.00 mm, vias 1 -> 0
- net /PWR_LINE_12V: track 22.3 -> 0.00 mm, vias 1 -> 0
- net /IRQ: track 20.9 -> 0.00 mm
- net /RST: track 20.9 -> 0.00 mm, vias 1 -> 0
- net /SDA: track 20.8 -> 0.00 mm
- net /SCL: track 20.8 -> 0.00 mm, vias 1 -> 0
- net +12V: track 119.3 -> 131.7 mm
- net +3V3: track 68.0 -> 62.1 mm, vias 4 -> 3
- net +5V: track 63.3 -> 59.3 mm, vias 0 -> 1
- net Net-(U2-LX): track 22.6 -> 21.6 mm
- net Net-(U1-LX): track 22.6 -> 21.6 mm
- net Net-(U2-BST): track 3.66 -> 2.80 mm
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Other:
- outline, holes or cut-outs redrawn
