File: board/t80-psu12.kicad_sch (KiCad schematic)
At the start: 28 parts

Commit message: WIP
Parts:
- removed NT1 (x5): NetTie_2, symbol Device:NetTie_2
- removed X1 (x2): ~, symbol t80:t80-pin-header
- added X1: ~, symbol t80:t80-pin-header
Connections:
- net +3V3: now also X1.4 (3V3)
- net +5V: now also X1.8 (5V)
- net GND: now also X1.1 (GND), X1.7 (GND)
- no-connect marks 0 -> 4
